Commit message: gazebo hw and controller connect

File: barrett_control/barrett_model/models/arm.urdf.xacro (robot description, xacro)
@@ -26,26 +26,4 @@
   <xacro:include filename="$(find barrett_model)/models/common.urdf.xacro"/>
   <xacro:include filename="$(find barrett_model)/models/components.urdf.xacro"/>
-  <xacro:macro name="wam_7dof" params="prefix parent_link xyz rpy">
-    <xacro:wam prefix="${prefix}" parent_link="${parent_link}" xyz="${xyz}" rpy="${rpy}"/>
-    <xacro:wam_wrist_left prefix="${prefix}"/>
-    <xacro:wam_wrist_palm_stump prefix="${prefix}"/>
-  </xacro:macro>
-  <xacro:macro name="wam_4dof" params="prefix parent_link xyz rpy">
-    <xacro:wam prefix="${prefix}" parent_link="${parent_link}" xyz="${xyz}" rpy="${rpy}"/>
-    <xacro:wam_stump prefix="${prefix}"/>
-  </xacro:macro>
-  <!-- upper arm only -->
-  <xacro:macro name="wam" params="prefix parent_link xyz rpy">
-    <xacro:wam_base prefix="${prefix}" parent_link="${parent_link}" xyz="${xyz}" rpy="${rpy}"/>
-    <xacro:wam_shoulder_yaw prefix="${prefix}" rpy="0 0 ${PI/2}" />
-    <xacro:wam_shoulder_pitch prefix="${prefix}" rpy="-${PI/2} ${PI/2} 0"/>
-    <xacro:wam_upper_arm prefix="${prefix}"/>
-  </xacro:macro>
-  <xacro:macro name="wam_right" params="prefix parent_link xyz rpy">
-    <xacro:wam_base prefix="${prefix}" parent_link="${parent_link}" xyz="${xyz}" rpy="${rpy}"/>
-    <xacro:wam_shoulder_yaw prefix="${prefix}" rpy="0 0 0" />
-    <xacro:wam_shoulder_pitch prefix="${prefix}" rpy="0 0 0"/>
-    <xacro:wam_upper_arm prefix="${prefix}" rpy="0 0 0"/>
-  </xacro:macro>
   <xacro:macro name="wam_left" params="prefix parent_link xyz rpy">
     <xacro:wam_base prefix="${prefix}" parent_link="${parent_link}" xyz="${xyz}" rpy="${rpy}"/>
@@ -55,4 +33,5 @@
   </xacro:macro>
   <!-- forearm with actuation "wrist" -->
+  <!--
   <xacro:macro name="wam_wrist_right" params="prefix">
     <xacro:wam_forearm prefix="${prefix}"/>
@@ -61,4 +40,5 @@
     <xacro:wam_palm prefix="${prefix}" rpy="${PI/2} -${PI/2} 0"/>
   </xacro:macro>
+  -->
   <xacro:macro name="wam_wrist_left" params="prefix">
     <xacro:wam_forearm prefix="${prefix}"/>

File: barrett_control/barrett_model/models/components.urdf.xacro (robot description, xacro)
@@ -24,7 +24,9 @@
 -->
 <robot xmlns:xacro="http://ros.org/wiki/xacro">
-  <xacro:include filename="$(find barrett_model)/models/hand.urdf.xacro"/>
+  <!-- <xacro:include filename="$(find barrett_model)/models/hand.urdf.xacro"/> -->
   <xacro:include filename="$(find barrett_model)/models/common.urdf.xacro"/>
   <xacro:property name="b" value="0.5"/>
+  <xacro:include filename="$(find barrett_model)/robots/wam7_bhand.transmission.xacro"/>
+  <xacro:include filename="$(find barrett_model)/robots/wam7_bhand.gazebo.xacro"/>
   <!-- Upper arm macros -->
   <xacro:macro name="wam_base" params="prefix parent_link xyz rpy">
@@ -64,5 +66,5 @@
       <origin xyz="0 0 0.346" rpy="${rpy}"/>
       <axis xyz="0 0 1"/>
-      <limit effort="60" lower="-2.6" upper="2.6" velocity="2.0"/>
+      <limit effort="25" lower="-2.6" upper="2.6" velocity="2.0"/>
       <dynamics damping="${1.8*b}" friction="0"/>
     </joint>
@@ -98,7 +100,7 @@
       <parent link="${prefix}/shoulder_yaw_link"/>
       <child link="${prefix}/shoulder_pitch_link"/>
-      <origin xyz="0 0 0" rpy="${rpy}"/>
-      <axis xyz="0 1 0"/>
-      <limit effort="60" lower="-2.0" upper="2.0" velocity="2.0"/>
+      <origin xyz="0 0 0" rpy="${-PI/2} 0 0"/>
+      <axis xyz="0 0 1"/>
+      <limit effort="20" lower="-2.0" upper="2.0" velocity="2.0"/>
       <dynamics damping="${0.5*b}" friction="0"/>
     </joint>
@@ -134,7 +136,7 @@
       <parent link="${prefix}/shoulder_pitch_link"/>
       <child link="${prefix}/upper_arm_link"/>
-      <origin xyz="0 0 0" rpy="${rpy}"/>
-      <axis xyz="0 0 1"/>
-      <limit effort="45" lower="-2.8" upper="2.8" velocity="2.0"/>
+      <origin xyz="0 0 0" rpy="${PI/2} 0 0"/>
+      <axis xyz="0 0 1"/>
+      <limit effort="15" lower="-2.8" upper="2.8" velocity="2.0"/>
       <dynamics damping="${1.5*b}" friction="0"/>
     </joint>
@@ -173,5 +175,5 @@
       <origin xyz="0.045 0 0.55" rpy="${-PI/2} 0 0"/>
       <axis xyz="0 0 1"/>
-      <limit effort="30" lower="-0.9" upper="${PI}" velocity="2.00"/>
+      <limit effort="15" lower="-0.9" upper="${PI}" velocity="2.00"/>
       <dynamics damping="${0.8*b}" friction="0"/>
     </joint>
@@ -224,5 +226,5 @@
       <origin xyz="-0.045 -0.3 0" rpy="${rpy}"/>
       <axis xyz="0 0 1"/>
-      <limit effort="10" lower="-4.76" upper="1.24" velocity="2.0"/>
+      <limit effort="5" lower="-4.76" upper="1.24" velocity="2.0"/>
       <dynamics damping="${0.5*b}" friction="0"/>
     </joint>
@@ -261,5 +263,5 @@
       <origin xyz="0 0 0" rpy="${-PI/2} 0 0"/>
       <axis xyz="0 0 1"/>
-      <limit effort="10" lower="-1.6" upper="1.6" velocity="2.00"/>
+      <limit effort="5" lower="-1.6" upper="1.6" velocity="2.00"/>
       <dynamics damping="${0.1*b}" friction="0"/>
     </joint>
@@ -296,7 +298,7 @@
       <parent link="${prefix}/wrist_pitch_link"/>
       <child link="${prefix}/wrist_palm_link"/>
-      <origin xyz="0 0 0" rpy="${rpy}"/>
-      <axis xyz="0 0 1"/>
-      <limit effort="10" lower="-3.0" upper="3.0" velocity="2.00"/><!-- 2.95 is a limit taken in from 3 due to saftey and differences between arms. -->
+      <origin xyz="0 0 0" rpy="${PI/2} 0 0"/>
+      <axis xyz="0 0 1"/>
+      <limit effort="5" lower="-3.0" upper="3.0" velocity="2.00"/><!-- 2.95 is a limit taken in from 3 due to saftey and differences between arms. -->
       <dynamics damping="${0.1*b}" friction="0"/>
     </joint>

File: barrett_control/barrett_model/robots/wam7_bhand.urdf.xacro (robot description, xacro)
@@ -4,4 +4,6 @@
   <!-- Includea all the WAM stuff -->
   <xacro:include filename="$(find barrett_model)/models/wam_top.urdf.xacro"/>
+  <xacro:include filename="$(find barrett_model)/robots/wam7_bhand.transmission.xacro"/>
+  <xacro:include filename="$(find barrett_model)/robots/wam7_bhand.gazebo.xacro"/>
   <!-- Root link is in the world frame-->
   <xacro:property name="width" value="0.0889" />
@@ -13,4 +15,12 @@
       </geometry>
     </visual>
+    <inertial>
+        <origin xyz="0 0 0" />
+        <mass value="1" />
+        <inertia
+          ixx="0.1" ixy="0"   ixz="0"
+                  iyy="0.1"   iyz="0"
+                            izz="0.1" />
+    </inertial>
   </link>
   <link name="rack2">
@@ -21,4 +31,12 @@
       <origin rpy="0 0 1.57075" xyz="0 0 0"/>
     </visual>
+    <inertial>
+        <origin xyz="0 0 0" />
+        <mass value="1" />
+        <inertia
+          ixx="0.1" ixy="0"   ixz="0"
+                  iyy="0.1"   iyz="0"
+                            izz="0.1" />
+    </inertial>
   </link>
   <link name="rack3">
@@ -29,4 +47,12 @@
       <origin rpy="0 0 1.57075" xyz="0 0 0"/>
     </visual>
+    <inertial>
+        <origin xyz="0 0 0" />
+        <mass value="1" />
+        <inertia
+          ixx="0.1" ixy="0"   ixz="0"
+                  iyy="0.1"   iyz="0"
+                            izz="0.1" />
+    </inertial>
   </link>
   <link name="rack4">
@@ -37,4 +63,12 @@
       <origin rpy="0 0 1.57075" xyz="0 0 0"/>
     </visual>
+    <inertial>
+        <origin xyz="0 0 0" />
+        <mass value="1" />
+        <inertia
+          ixx="0.1" ixy="0"   ixz="0"
+                  iyy="0.1"   iyz="0"
+                            izz="0.1" />
+    </inertial>
   </link>
   <link name="rack5">
@@ -45,4 +79,12 @@
       <origin rpy="0 1.57075 0" xyz="0 0 0.9525"/>
     </visual>
+    <inertial>
+        <origin xyz="0 0 0" />
+        <mass value="1" />
+        <inertia
+          ixx="0.1" ixy="0"   ixz="0"
+                  iyy="0.1"   iyz="0"
+                            izz="0.1" />
+      </inertial>
   </link>
   <link name="rack6">
@@ -53,7 +95,33 @@
       <origin rpy="0 0 0" xyz="0 0 0"/>
     </visual>
+    <inertial>
+        <origin xyz="0 0 0" />
+        <mass value="1" />
+        <inertia
+          ixx="0.1" ixy="0"   ixz="0"
+                  iyy="0.1"   iyz="0"
+                            izz="0.1" />
+    </inertial>
   </link>
-  <link name ="left_wam_rack" />
-  <link name ="right_wam_rack" />
+  <link name ="left_wam_rack">
+    <inertial>
+        <origin xyz="0 0 0" />
+        <mass value="1" />
+        <inertia
+          ixx="0.1" ixy="0"   ixz="0"
+                  iyy="0.1"   iyz="0"
+                            izz="0.1" />
+    </inertial>
+  </link>
+  <link name ="right_wam_rack">
+    <inertial>
+        <origin xyz="0 0 0" />
+        <mass value="1" />
+        <inertia
+          ixx="0.1" ixy="0"   ixz="0"
+                  iyy="0.1"   iyz="0"
+                            izz="0.1" />
+     </inertial>
+  </link>
   <joint name="rack1_to_rack2" type="fixed">
     <parent link="rack1"/>
@@ -99,4 +167,7 @@
   <xacro:wam_left prefix="left_wam" parent_link="left_wam_rack" xyz="0.0 0.0 0" rpy="-1.57075 ${-PI} 0" />
   <xacro:wam_wrist_left prefix="left_wam"/>
+  <!-- gazebo stuff -->
+  <xacro:wam7_bhand_gazebo prefix="left_wam" name="barrett_hw"/>
+  <xacro:wam7_bhand_transmission prefix="left_wam" name="barrett_hw"/>
   <!-- <xacro:bhand prefix="left_wam/bhand" parent_link="left_wam/wrist_palm_link" xyz="0 0 0.06" rpy="0 0 0"/> -->
 </robot>

Commit message: impedance controller

File: barrett_control/barrett_model/models/arm.urdf.xacro (robot description, xacro)
@@ -33,12 +33,12 @@
   </xacro:macro>
   <!-- forearm with actuation "wrist" -->
-  <!--
   <xacro:macro name="wam_wrist_right" params="prefix">
-    <xacro:wam_forearm prefix="${prefix}"/>
+    <!-- <xacro:wam_forearm prefix="${prefix}"/> -->
+    <!--
     <xacro:wam_wrist_yaw prefix="${prefix}" rpy="${PI/2} 0 0"/>
     <xacro:wam_wrist_pitch prefix="${prefix}"/>
     <xacro:wam_palm prefix="${prefix}" rpy="${PI/2} -${PI/2} 0"/>
+    -->
   </xacro:macro>
-  -->
   <xacro:macro name="wam_wrist_left" params="prefix">
     <xacro:wam_forearm prefix="${prefix}"/>

File: barrett_control/barrett_model/models/components.urdf.xacro (robot description, xacro)
@@ -51,4 +51,5 @@
         <geometry>
           <mesh filename="${models_path}/sw_meshes/base_link_convex.dae"/>
+          <!-- <mesh filename="package://barrett_model/meshes/wambase.stl" /> -->
         </geometry>
       </visual>
@@ -56,4 +57,5 @@
         <geometry>
           <mesh filename="${models_path}/sw_meshes/base_link_convex.dae"/>
+          <!-- <mesh filename="package://barrett_model/meshes/wambase.stl" /> -->
         </geometry>
       </collision>
@@ -87,4 +89,5 @@
         <geometry>
           <mesh filename="${models_path}/sw_meshes/shoulder_link_convex_decomposition.dae"/>
+          <!-- <mesh filename="package://barrett_model/meshes/wam1.stl" /> -->
         </geometry>
       </visual>
@@ -92,4 +95,5 @@
         <geometry>
           <mesh filename="${models_path}/sw_meshes/shoulder_link_convex_decomposition.dae"/>
+          <!-- <mesh filename="package://barrett_model/meshes/wam1.stl" /> -->
         </geometry>
       </collision>
@@ -115,4 +119,5 @@
         <geometry>
           <mesh filename="${models_path}/sw_meshes/shoulder_pitch_link_convex.dae"/>
+          <!-- <mesh filename="package://barrett_model/meshes/wam2.stl" /> -->
         </geometry>
       </visual>
@@ -128,4 +133,5 @@
         <geometry>
           <mesh filename="${models_path}/sw_meshes/shoulder_pitch_link_convex.dae"/>
+          <!-- <mesh filename="package://barrett_model/meshes/wam2.stl" /> -->
         </geometry>
       </collision>
@@ -159,4 +165,5 @@
         <geometry>
           <mesh filename="${models_path}/sw_meshes/upper_arm_link_convex_decomposition.dae"/>
+          <!-- <mesh filename="package://barrett_model/meshes/wam3.stl" /> -->
         </geometry>
       </visual>
@@ -164,4 +171,5 @@
         <geometry>
           <mesh filename="${models_path}/sw_meshes/upper_arm_link_convex_decomposition.dae"/>
+          <!-- <mesh filename="package://barrett_model/meshes/wam3.stl" /> -->
         </geometry>
       </collision>
@@ -196,4 +204,5 @@
         <geometry>
           <mesh filename="${models_path}/sw_meshes/elbow_link_convex.dae"/>
+          <!-- <mesh filename="package://barrett_model/meshes/wam4.stl" /> -->
         </geometry>
       </visual>
@@ -201,6 +210,8 @@
         <geometry>
           <mesh filename="${models_path}/sw_meshes/elbow_link_convex.dae"/>
-        </geometry>
-      </collision>
+          <!-- <mesh filename="package://barrett_model/meshes/wam4.stl" /> -->
+        </geometry>
+      </collision>
+      <!--
       <visual>
         <material name="WAMGrey">
@@ -212,4 +223,5 @@
         </geometry>
       </visual>
+      -->
       <collision>
         <origin xyz="-0.045 -0.0730 0" rpy="${PI/2} 0 0" />
@@ -247,4 +259,5 @@
         <geometry>
           <mesh filename="${models_path}/sw_meshes/wrist_yaw_link_convex_decomposition.dae"/>
+          <!-- <mesh filename="package://barrett_model/meshes/wam5.stl" /> -->
         </geometry>
       </visual>
@@ -253,4 +266,5 @@
         <geometry>
           <mesh filename="${models_path}/sw_meshes/wrist_yaw_link_convex_decomposition.dae"/>
+          <!-- <mesh filename="package://barrett_model/meshes/wam5.stl" /> -->
         </geometry>
       </collision>
@@ -284,4 +298,5 @@
         <geometry>
           <mesh filename="${models_path}/sw_meshes/wrist_pitch_link_convex_decomposition.dae"/>
+          <!-- <mesh filename="package://barrett_model/meshes/wam6.stl" /> -->
         </geometry>
       </visual>
@@ -289,4 +304,5 @@
         <geometry>
           <mesh filename="${models_path}/sw_meshes/wrist_pitch_link_convex_decomposition.dae"/>
+          <!-- <mesh filename="package://barrett_model/meshes/wam6.stl" /> -->
         </geometry>
       </collision>
@@ -321,4 +337,5 @@
         <geometry>
           <mesh filename="${models_path}/sw_meshes/wrist_palm_link_convex.dae"/>
+          <!--<mesh filename="package://barrett_model/meshes/wam7.stl" /> -->
         </geometry>
       </visual>
@@ -327,4 +344,5 @@
         <geometry>
           <mesh filename="${models_path}/sw_meshes/wrist_palm_link_convex.dae"/>
+          <!-- <mesh filename="package://barrett_model/meshes/wam7.stl" /> -->
         </geometry>
       </collision>
@@ -373,5 +391,5 @@
         <!--<origin xyz="0 0 0" rpy="-${PI} 0 0" />-->
         <!--<geometry>-->
-          <!--<mesh filename="${models_path}/meshes/wamForeArmLink4.DAE"/>-->
+          <!--<mesh filename="${models_path}/meshes/wamForeArmLink4.dae"/>-->
         <!--</geometry>-->
       <!--</visual>-->
@@ -379,5 +397,5 @@
         <!--<origin xyz="0 0 0" rpy="-${PI} 0 0" />-->
         <!--<geometry>-->
-          <!--<mesh filename="${models_path}/meshes/wamForeArmLink4.stl"/>-->
+          <!--<mesh filename="${models_path}/meshes/wamForeArmLink4.dae"/>-->
         <!--</geometry>-->
       <!--</collision>-->
@@ -408,5 +426,5 @@
         <!--<origin xyz="0 0.02711 0" rpy="${PI} 0 0" />-->
         <!--<geometry>-->
-          <!--<mesh filename="${models_path}/meshes/wamUpperWristYawLink.DAE"/>-->
+          <!--<mesh filename="${models_path}/meshes/wamUpperWristYawLink.dae"/>-->
         <!--</geometry>-->
       <!--</visual>-->
@@ -414,5 +432,5 @@
         <!--<origin xyz="0 0.02711 0" rpy="${PI} 0 0" />-->
         <!--<geometry>-->
-          <!--<mesh filename="${models_path}/meshes/wamUpperWristYawLink5.stl"/>-->
+          <!--<mesh filename="${models_path}/meshes/wamUpperWristYawLink5.dae"/>-->
         <!--</geometry>-->
       <!--</collision>-->
@@ -444,5 +462,5 @@
         <!--<origin xyz="0 0 0" rpy="0 0 0" />-->
         <!--<geometry>-->
-          <!--<mesh filename="${models_path}/meshes/forceTorqueSensor.DAE"/>-->
+          <!--<mesh filename="${models_path}/meshes/forceTorqueSensor.dae"/>-->
         <!--</geometry>-->
       <!--</visual>-->
@@ -450,5 +468,5 @@
         <!--<origin xyz="0 0 0" rpy="0 0 0" />-->
         <!--<geometry>-->
-          <!--<mesh filename="${models_path}/meshes/forceTorqueSensor.stl"/>-->
+          <!--<mesh filename="${models_path}/meshes/forceTorqueSensor.dae"/>-->
         <!--</geometry>-->
       <!--</collision>-->

File: barrett_control/barrett_model/robots/wam7_bhand.gazebo.xacro (robot description, xacro)
@@ -9,33 +9,33 @@
 		<gazebo reference="${prefix}/base_link">
 			<gravity>true</gravity>
-			<material>Gazebo/Orange</material>
+			<material>Gazebo/Grey</material>
 		</gazebo>
 		<gazebo reference="${prefix}/shoulder_yaw_link">
 			<gravity>true</gravity>
-			<material>Gazebo/Orange</material>
+			<material>Gazebo/Grey</material>
 		</gazebo>
 		<gazebo reference="${prefix}/shoulder_pitch_link">
 			<gravity>true</gravity>
-			<material>Gazebo/Orange</material>
+			<material>Gazebo/Grey</material>
 		</gazebo>
 		<gazebo reference="${prefix}/upper_arm_link">
 			<gravity>true</gravity>
-			<material>Gazebo/Orange</material>
+			<material>Gazebo/Grey</material>
 		</gazebo>
 		<gazebo reference="${prefix}/forearm_link">
 			<gravity>true</gravity>
-			<material>Gazebo/Orange</material>
+			<material>Gazebo/Grey</material>
 		</gazebo>
 		<gazebo reference="${prefix}/wrist_yaw_link">
 			<gravity>true</gravity>
-			<material>Gazebo/Orange</material>
+			<material>Gazebo/Grey</material>
 		</gazebo>
 		<gazebo reference="${prefix}/wrist_pitch_link">
 			<gravity>true</gravity>
-			<material>Gazebo/Orange</material>
+			<material>Gazebo/Grey</material>
 		</gazebo>
 		<gazebo reference="${prefix}/wrist_palm_link">
 			<gravity>true</gravity>
-			<material>Gazebo/Grey</material>
+			<material>Gazebo/Red</material>
 		</gazebo>
 	</xacro:macro>

File: barrett_control/barrett_model/robots/wam7_bhand.urdf.xacro (robot description, xacro)
@@ -9,4 +9,9 @@
   <xacro:property name="width" value="0.0889" />
   <xacro:property name="height" value="0.0492125" />
+  <link name="world"/>
+  <joint name="fixed" type="fixed">
+    <parent link="world"/>
+    <child link="rack1"/>
+  </joint>
   <link name="rack1">
     <visual>
@@ -167,7 +172,7 @@
   <xacro:wam_left prefix="left_wam" parent_link="left_wam_rack" xyz="0.0 0.0 0" rpy="-1.57075 ${-PI} 0" />
   <xacro:wam_wrist_left prefix="left_wam"/>
+  <!-- <xacro:bhand prefix="left_wam/bhand" parent_link="left_wam/wrist_palm_link" xyz="0 0 0.06" rpy="0 0 0"/> -->
   <!-- gazebo stuff -->
   <xacro:wam7_bhand_gazebo prefix="left_wam" name="barrett_hw"/>
   <xacro:wam7_bhand_transmission prefix="left_wam" name="barrett_hw"/>
-  <!-- <xacro:bhand prefix="left_wam/bhand" parent_link="left_wam/wrist_palm_link" xyz="0 0 0.06" rpy="0 0 0"/> -->
 </robot>
