Commit message: pid brings the wam to the desired home position

File: barrett_control/barrett_model/models/components.urdf.xacro (robot description, xacro)
@@ -69,5 +69,5 @@
       <axis xyz="0 0 1"/>
       <limit effort="25" lower="-2.6" upper="2.6" velocity="2.0"/>
-      <dynamics damping="${1.8*b}" friction="0"/>
+      <dynamics damping="${1.8*b}" friction="10"/>
     </joint>
     <gazebo reference="${prefix}/base_yaw_joint">
@@ -107,5 +107,5 @@
       <axis xyz="0 0 1"/>
       <limit effort="20" lower="-2.0" upper="2.0" velocity="2.0"/>
-      <dynamics damping="${0.5*b}" friction="0"/>
+      <dynamics damping="${0.5*b}" friction="10"/>
     </joint>
     <gazebo reference="${prefix}/shoulder_pitch_joint">
@@ -145,5 +145,5 @@
       <axis xyz="0 0 1"/>
       <limit effort="15" lower="-2.8" upper="2.8" velocity="2.0"/>
-      <dynamics damping="${1.5*b}" friction="0"/>
+      <dynamics damping="${1.5*b}" friction="10"/>
     </joint>
     <gazebo reference="${prefix}/shoulder_yaw_joint">
@@ -184,5 +184,5 @@
       <axis xyz="0 0 1"/>
       <limit effort="15" lower="-0.9" upper="${PI}" velocity="2.00"/>
-      <dynamics damping="${0.8*b}" friction="0"/>
+      <dynamics damping="${0.8*b}" friction="10"/>
     </joint>
     <gazebo reference="${prefix}/elbow_pitch_joint">
@@ -213,5 +213,4 @@
         </geometry>
       </collision>
-      <!--
       <visual>
         <material name="WAMGrey">
@@ -223,5 +222,4 @@
         </geometry>
       </visual>
-      -->
       <collision>
         <origin xyz="-0.045 -0.0730 0" rpy="${PI/2} 0 0" />
@@ -239,5 +237,5 @@
       <axis xyz="0 0 1"/>
       <limit effort="5" lower="-4.76" upper="1.24" velocity="2.0"/>
-      <dynamics damping="${0.5*b}" friction="0"/>
+      <dynamics damping="${0.5*b}" friction="10"/>
     </joint>
     <gazebo reference="${prefix}/wrist_yaw_joint">
@@ -278,5 +276,5 @@
       <axis xyz="0 0 1"/>
       <limit effort="5" lower="-1.6" upper="1.6" velocity="2.00"/>
-      <dynamics damping="${0.1*b}" friction="0"/>
+      <dynamics damping="${0.1*b}" friction="10"/>
     </joint>
     <gazebo reference="${prefix}/wrist_pitch_joint">
@@ -317,5 +315,5 @@
       <axis xyz="0 0 1"/>
       <limit effort="5" lower="-3.0" upper="3.0" velocity="2.00"/><!-- 2.95 is a limit taken in from 3 due to saftey and differences between arms. -->
-      <dynamics damping="${0.1*b}" friction="0"/>
+      <dynamics damping="${0.1*b}" friction="10"/>
     </joint>
     <gazebo reference="${prefix}/palm_yaw_joint">

Commit message: bunch of new stuff

File: barrett_control/barrett_model/models/components.urdf.xacro (robot description, xacro)
@@ -69,5 +69,5 @@
       <axis xyz="0 0 1"/>
       <limit effort="25" lower="-2.6" upper="2.6" velocity="2.0"/>
-      <dynamics damping="${1.8*b}" friction="10"/>
+      <dynamics damping="${1.8*b}" friction="0"/>
     </joint>
     <gazebo reference="${prefix}/base_yaw_joint">
@@ -106,6 +106,6 @@
       <origin xyz="0 0 0" rpy="${-PI/2} 0 0"/>
       <axis xyz="0 0 1"/>
-      <limit effort="20" lower="-2.0" upper="2.0" velocity="2.0"/>
-      <dynamics damping="${0.5*b}" friction="10"/>
+      <limit effort="30" lower="-2.0" upper="2.0" velocity="2.0"/>
+      <dynamics damping="${0.5*b}" friction="0"/>
     </joint>
     <gazebo reference="${prefix}/shoulder_pitch_joint">
@@ -145,5 +145,5 @@
       <axis xyz="0 0 1"/>
       <limit effort="15" lower="-2.8" upper="2.8" velocity="2.0"/>
-      <dynamics damping="${1.5*b}" friction="10"/>
+      <dynamics damping="${1.5*b}" friction="0"/>
     </joint>
     <gazebo reference="${prefix}/shoulder_yaw_joint">
@@ -184,5 +184,5 @@
       <axis xyz="0 0 1"/>
       <limit effort="15" lower="-0.9" upper="${PI}" velocity="2.00"/>
-      <dynamics damping="${0.8*b}" friction="10"/>
+      <dynamics damping="${0.8*b}" friction="0"/>
     </joint>
     <gazebo reference="${prefix}/elbow_pitch_joint">
@@ -237,5 +237,5 @@
       <axis xyz="0 0 1"/>
       <limit effort="5" lower="-4.76" upper="1.24" velocity="2.0"/>
-      <dynamics damping="${0.5*b}" friction="10"/>
+      <dynamics damping="${0.5*b}" friction="0"/>
     </joint>
     <gazebo reference="${prefix}/wrist_yaw_joint">
@@ -276,5 +276,5 @@
       <axis xyz="0 0 1"/>
       <limit effort="5" lower="-1.6" upper="1.6" velocity="2.00"/>
-      <dynamics damping="${0.1*b}" friction="10"/>
+      <dynamics damping="${0.1*b}" friction="0"/>
     </joint>
     <gazebo reference="${prefix}/wrist_pitch_joint">
@@ -315,5 +315,5 @@
       <axis xyz="0 0 1"/>
       <limit effort="5" lower="-3.0" upper="3.0" velocity="2.00"/><!-- 2.95 is a limit taken in from 3 due to saftey and differences between arms. -->
-      <dynamics damping="${0.1*b}" friction="10"/>
+      <dynamics damping="${0.1*b}" friction="0"/>
     </joint>
     <gazebo reference="${prefix}/palm_yaw_joint">
