Commit message: osc less weird?

File: barrett_control/barrett_model/models/components_copy.urdf.xacro (robot description, xacro)
@@ -68,5 +68,5 @@
       <origin xyz="0 0 0.346" rpy="${rpy}"/>
       <axis xyz="0 0 1"/>
-      <limit effort="40" lower="-2.6" upper="2.6" velocity="2.0"/>
+      <limit effort="25" lower="-2.6" upper="2.6" velocity="2.0"/>
       <dynamics damping="${1.8*b}" friction="1"/>
     </joint>
@@ -76,10 +76,10 @@
     <link name="${prefix}/shoulder_yaw_link" >
       <inertial>
-        <origin xyz="-.00443422 -.00066489 -0.1289039 " />
+        <origin xyz="-.00443422 0.1289039 -.00066489  " />
         <mass value="10.7677" />
         <inertia
-          ixx=".13488033"  ixy="-0.00012485"   ixz="0.00213041"
-                           iyy=".09046330"    iyz="-.00068555"
-                                              izz=".11328369" />
+          ixx=".13488033"  ixy="-0.00213041"   ixz="-0.00012485"
+                           iyy=".11328369"    iyz=".00068555"
+                                              izz=".09046330" />
       </inertial>
       <visual>
@@ -106,5 +106,5 @@
       <origin xyz="0 0 0" rpy="${-PI/2} 0 0"/>
       <axis xyz="0 0 1"/>
-      <limit effort="40" lower="-2.0" upper="2.0" velocity="2.0"/>
+      <limit effort="30" lower="-2.0" upper="2.0" velocity="2.0"/>
       <dynamics damping="${0.5*b}" friction="1"/>
     </joint>
@@ -123,10 +123,10 @@
       </visual>
       <inertial>
-        <origin xyz="-.00236981 -.01542114 .03105614 "/>
+        <origin xyz="-.00236981 .03105614 .01542114 "/>
         <mass value="3.87493756" />
         <inertia
-          ixx="0.02140958"  ixy="-0.00002461"  ixz="0.00027172"
-                            iyy="0.015589060"  iyz="0.0018192"
-                                               izz="0.01377875" />
+          ixx="0.02140958"  ixy="0.00027172"  ixz="0.00002461"
+                            iyy="0.01377875"  iyz="-0.0018192"
+                                               izz="0.015589060" />
       </inertial>
       <collision>
@@ -144,5 +144,5 @@
       <origin xyz="0 0 0" rpy="${PI/2} 0 0"/>
       <axis xyz="0 0 1"/>
-      <limit effort="40" lower="-2.8" upper="2.8" velocity="2.0"/>
+      <limit effort="15" lower="-2.8" upper="2.8" velocity="2.0"/>
       <dynamics damping="${1.5*b}" friction="1"/>
     </joint>
@@ -152,10 +152,10 @@
     <link name="${prefix}/upper_arm_link" >
       <inertial>
-        <origin xyz="0.00683258580000000 0.000033090000000 0.392492300000000" />
+        <origin xyz="0.00382658580000000 0.207512300000000 0.000033090000000" />
         <mass value="1.8023" />
         <inertia
-          ixx=".05911077"  ixy="-0.00000738"  ixz="-0.00249612"
-                           iyy="0.05927043"   iyz="0.00001767"
-                                              izz="0.0032455" />
+          ixx=".05911077"  ixy="-0.00249612"  ixz="0.00000738"
+                           iyy="0.0032455"   iyz="-0.00001767"
+                                              izz="0.05927043" />
       </inertial>
       <visual>
@@ -183,5 +183,5 @@
       <origin xyz="0.045 0 0.55" rpy="${-PI/2} 0 0"/>
       <axis xyz="0 0 1"/>
-      <limit effort="40" lower="-0.9" upper="${PI}" velocity="2.00"/>
+      <limit effort="15" lower="-0.9" upper="${PI}" velocity="2.00"/>
       <dynamics damping="${0.8*b}" friction="1"/>
     </joint>
@@ -192,9 +192,9 @@
       <inertial>
         <mass value="2.17266212" />
-        <origin xyz="-0.04001488 -.14271662 -.00022942 " rpy="0 0 0" />
-        <inertia
-          ixx="0.01491672" ixy="0.001506040000000" ixz="0.000017410000000"
-                           iyy="0.002944630000000" iyz="0.000021090000000"
-                                                   izz="0.014829880000000" />
+        <origin xyz="0.00553408 0.00006822 0.11927695" rpy="0 0 0" />
+        <inertia
+          ixx="0.01067491" ixy="0.00004503" ixz="-0.00135557"
+                           iyy="0.01058659" iyz="-0.00011002"
+                                                   izz="0.00282036" />
       </inertial>
       <visual>
@@ -236,5 +236,5 @@
       <origin xyz="-0.045 -0.3 0" rpy="${rpy}"/>
       <axis xyz="0 0 1"/>
-      <limit effort="40" lower="-4.76" upper="1.24" velocity="2.0"/>
+      <limit effort="5" lower="-4.76" upper="1.24" velocity="2.0"/>
       <dynamics damping="${0.5*b}" friction="1"/>
     </joint>
@@ -244,9 +244,9 @@
     <link name="${prefix}/wrist_yaw_link" >
       <inertial>
-        <origin xyz="0.00008921 0.00435824 -0.00511217 " />
+        <origin xyz="0.00005483 0.02886286 0.00148493 " />
         <mass value="0.35655692" />
-        <inertia  ixx="0.00005029" ixy="0.00000020"  ixz="0.00007582"
-          iyy="0.00007582"  iyz="-0.00000359"
-          izz="0.00006270" />
+        <inertia  ixx="0.00037112" ixy="-0.00000008"  ixz="-0.00000003"
+          iyy="0.00019434"  iyz="-0.00001613"
+          izz="0.00038209" />
       </inertial>
       <visual>
@@ -275,5 +275,5 @@
       <origin xyz="0 0 0" rpy="${-PI/2} 0 0"/>
       <axis xyz="0 0 1"/>
-      <limit effort="40" lower="-1.6" upper="1.6" velocity="2.00"/>
+      <limit effort="5" lower="-1.6" upper="1.6" velocity="2.00"/>
       <dynamics damping="${0.1*b}" friction="1"/>
     </joint>
@@ -283,10 +283,10 @@
     <link name="${prefix}/wrist_pitch_link" >
       <inertial>
-        <origin xyz="-0.00012262 -0.02468336 -0.01703194 " rpy="0 0 0" />
+        <origin xyz="-0.00005923 -0.01686123 0.02419052" rpy="0 0 0" />
         <mass value="0.40915886" />
         <inertia
-          ixx="0.00055516"  ixy="0.00000061"  ixz="-0.00000074"
-          iyy="0.00024367"  iyz="-0.00004590"
-          izz="0.00045358" />
+          ixx="0.00054889"  ixy="0.00000019"  ixz="-0.00000010"
+          iyy="0.00023846"  iyz="-0.00004430"
+          izz="0.00045133" />
       </inertial>
       <visual>
@@ -314,5 +314,5 @@
       <origin xyz="0 0 0" rpy="${PI/2} 0 0"/>
       <axis xyz="0 0 1"/>
-      <limit effort="40" lower="-3.0" upper="3.0" velocity="2.00"/><!-- 2.95 is a limit taken in from 3 due to saftey and differences between arms. -->
+      <limit effort="5" lower="-3.0" upper="3.0" velocity="2.00"/><!-- 2.95 is a limit taken in from 3 due to saftey and differences between arms. -->
       <dynamics damping="${0.1*b}" friction="1"/>
     </joint>
@@ -322,9 +322,9 @@
     <link name="${prefix}/wrist_palm_link" >
       <inertial>
-        <origin xyz="0.0 0.0 0.055" rpy="0 0 0" />
+        <origin xyz="0.00014836 0.00007252 -0.00335185" rpy="0 0 0" />
         <mass value="0.07548270" />
-        <inertia  ixx="0.00010859" ixy="0.00000000"  ixz="-0.00000000"
-          iyy="0.00020683"  iyz="-0.0000000"
-          izz="0.00010851" />
+        <inertia  ixx="0.00003911" ixy="0.00000019"  ixz="-0.00000000"
+          iyy="0.00003877"  iyz="-0.0000000"
+          izz="0.00007614" />
       </inertial>
       <visual>

File: barrett_control/lwr_description/model/kuka_lwr.gazebo.xacro (robot description, xacro)
@@ -3,5 +3,5 @@
 	<xacro:macro name="kuka_lwr_gazebo" params="name">
 		<gazebo>
-			<plugin name="${name}_lwr_hw_sim" filename="libbase_robot_hw_gazebo_plugin.so">
+			<plugin name="${name}_lwr_hw_sim" filename="libsim_robot_hw_gazebo_plugin.so">
 				<robotNamespace>${name}</robotNamespace>
 			</plugin>
@@ -37,5 +37,5 @@
 		<gazebo reference="${name}_7_link">
 			<gravity>true</gravity>
-			<material>Gazebo/Grey</material>
+			<material>Gazebo/Red</material>
 		</gazebo>
 	</xacro:macro>

File: barrett_control/lwr_description/model/kuka_lwr.urdf.xacro (robot description, xacro)
@@ -366,6 +366,6 @@
 			</collision>
 		</link>
-		<xacro:kuka_lwr_gazebo name="${name}"/>
-		<xacro:kuka_lwr_transmission name="${name}"/>
+		<xacro:kuka_lwr_gazebo name="sim_hw"/>
+		<xacro:kuka_lwr_transmission name="lwr"/>
 	</xacro:macro>
 </robot>

File: barrett_control/lwr_description/model/single_lwr_robot.urdf.xacro (robot description, xacro)
@@ -3,4 +3,9 @@
 	<!-- Include all models -->
 	<xacro:include filename="$(find lwr_description)/model/kuka_lwr.urdf.xacro"/>
+        <link name="world"/>
+          <joint name="fixed" type="fixed">
+          <parent link="world"/>
+          <child link="box1"/>
+        </joint>
 	<!-- and assemble your robot -->
 	<link name="box1">
